File: LinuxBoard KiCad/LinuxBoard.kicad_sch (KiCad schematic)
At the start: 0 parts

Commit message: Added F1C100s to Schematic
Parts:
- added IC1: F1C100S, QFN40P1000X1000X90-89N-D, symbol Linux Board Library:F1C100S
Changed lines of the file:
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@@
     (company "devTwins")
+  )
+  (symbol (lib_id "Linux Board Library:F1C100S") (at 106.68 62.23 0) (unit 1)
+    (in_bom yes) (on_board yes) (fields_autoplaced)
+    (property "Reference" "IC1" (id 0) (at 177.8 55.6512 0))
+    (property "Value" "F1C100S" (id 1) (at 177.8 58.1912 0))
+    (property "Footprint" "QFN40P1000X1000X90-89N-D" (id 2) (at 173.99 44.45 0)
+      (effects (font (size 1.27 1.27)) (justify left) hide)
+    )
+    (property "Datasheet" "https://linux-sunxi.org/images/b/ba/F1C100s_Datasheet_V1.0.pdf" (id 3) (at 173.99 46.99 0)
+      (effects (font (size 1.27 1.27)) (justify left) hide)
+    )
+    (property "Description" "F1C100s Processor" (id 4) (at 173.99 49.53 0)
+      (effects (font (size 1.27 1.27)) (justify left) hide)
+    )
+    (property "Height" "0.9" (id 5) (at 173.99 52.07 0)
+      (effects (font (size 1.27 1.27)) (justify left) hide)
+    )
+    (property "Manufacturer_Name" "Allwinner Technology" (id 6) (at 173.99 54.61 0)
+      (effects (font (size 1.27 1.27)) (justify left) hide)
+    )
+    (property "Manufacturer_Part_Number" "F1C100S" (id 7) (at 173.99 57.15 0)
+      (effects (font (size 1.27 1.27)) (justify left) hide)
+    )
+    (property "Mouser Part Number" "" (id 8) (at 173.99 59.69 0)
+      (effects (font (size 1.27 1.27)) (justify left) hide)
+    )
+    (property "Mouser Price/Stock" "" (id 9) (at 173.99 62.23 0)
+      (effects (font (size 1.27 1.27)) (justify left) hide)
+    )
+    (property "Arrow Part Number" "" (id 10) (at 173.99 64.77 0)
+      (effects (font (size 1.27 1.27)) (justify left) hide)
+    )
+    (property "Arrow Price/Stock" "" (id 11) (at 173.99 67.31 0)
+      (effects (font (size 1.27 1.27)) (justify left) hide)
+    )
+    (pin "1")
+    (pin "10")
+    (pin "11")
+    (pin "12")
+    (pin "13")
+    (pin "14")
+    (pin "15")
+    (pin "16")
+    (pin "17")
+    (pin "18")
+    (pin "19")
+    (pin "2")
+    (pin "20")
+    (pin "21")
+    (pin "22")
+    (pin "23")
+    (pin "24")
+    (pin "25")
+    (pin "26")
+    (pin "27")
+    (pin "28")
+    (pin "29")
+    (pin "3")
+    (pin "30")
+    (pin "31")
+    (pin "32")
+    (pin "33")
+    (pin "34")
+    (pin "35")
+    (pin "36")
+    (pin "37")
+    (pin "38")
+    (pin "39")
+    (pin "4")
+    (pin "40")
+    (pin "41")
+    (pin "42")
+    (pin "43")
+    (pin "44")
+    (pin "45")
+    (pin "46")
+    (pin "47")
+    (pin "48")
+    (pin "49")
+    (pin "5")
+    (pin "50")
+    (pin "51")
+    (pin "52")
+    (pin "53")
+    (pin "54")
+    (pin "55")
+    (pin "56")
+    (pin "57")
+    (pin "58")
+    (pin "59")
+    (pin "6")
+    (pin "60")
+    (pin "61")
+    (pin "62")
+    (pin "63")
+    (pin "64")
+    (pin "65")
+    (pin "66")
+    (pin "67")
+    (pin "68")
+    (pin "69")
+    (pin "7")
+    (pin "70")
+    (pin "71")
+    (pin "72")
+    (pin "73")
+    (pin "74")
+    (pin "75")
+    (pin "76")
+    (pin "77")
+    (pin "78")
+    (pin "79")
+    (pin "8")
+    (pin "80")
+    (pin "81")
+    (pin "82")
+    (pin "83")
+    (pin "84")
+    (pin "85")
+    (pin "86")
+    (pin "87")
+    (pin "88")
+    (pin "89")
+    (pin "9")
   )
   (sheet_instances
     (path "/" (page "1"))
   )
+  (symbol_instances
+    (path "/cc03413d-5116-45be-9c77-f360234077bd"
+      (reference "IC1") (unit 1) (value "F1C100S") (footprint "QFN40P1000X1000X90-89N-D")
+    )
+  )
 )
